File: Fake-Alarm/PCB/Fake Alarm.sch (EAGLE design)
At the start: 15 parts, among them IC1 NE555DG4, X3 009176003

Commit message: Remove the OLD
Parts:
- removed H1, H2, H3, H4: MOUNT-HOLE3.0, holes:MOUNT-HOLE3.0
- removed SS8550: (no value), zetex:PNPSOT89
- removed X3: 009176003, con-avx:009176003
- added C2: 10uF, rcl:C-EUC0805K
- added SV1: (no value), con-lstb:MA04-1
- added T1: (no value), zetex:PNPSOT23
- R4: value (none) -> 10k
Connections:
- net GND: now also C2.2, SV1.1
- net N$1: now also C2.1, T1.E; no longer SS8550.E
- net N$4: now also T1.C; no longer SS8550.C
- net N$5: now also SV1.2, T1.B; no longer SS8550.B, X3.1
- net N$8: now also SV1.3; no longer X3.2
- net N$9: now also SV1.4; no longer X3.3
Other:
- moved on the sheet: 1N5819, R4, R5
